File: schematic/unijoysticle.sch (EAGLE design)
At the start: 8 parts, among them CN1 External Battery, IC1 4066N, IC2 4066N, IC3 4066N, X1 Joy #1, X2 Joy #2

Commit message: fix: schematic & board fixed
Parts:
- CN1: value External Battery -> 3.3V - 9V; OC_NEWARK (none) -> unknown
- D1, ESP1, IC1, IC2, IC3: OC_NEWARK (none) -> unknown
- renumbered U$1 to ESP1
Connections:
- net N$24 renamed 5V
- removed net N$25: CN1.GND, ESP1.GND@1
- new net 3.3V: CN1.GND, CN1.GNDBREAK, ESP1.GND@1
- net N$13: now also IC3A.A; no longer IC2A.A
- net N$14: now also IC3B.A; no longer IC2B.A
- net N$15: now also IC3C.A; no longer IC2C.A
- net N$16: now also IC3D.A; no longer IC2D.A
- net N$17: now also IC2A.B; no longer IC3A.B
- net N$18: now also IC3A.B, IC3C.B, IC3D.B; no longer IC2A.B, IC2C.B, IC2D.B
- net N$19: now also IC2A.C; no longer IC3A.C
- net N$20: now also IC2B.C; no longer IC3B.C
- net N$21: now also IC2A.A; no longer IC3A.A
- net N$22: now also IC2B.A; no longer IC3B.A
- net N$5: now also IC3A.C; no longer IC2A.C
- net N$6: now also IC3B.C; no longer IC2B.C
- net N$7: now also IC3C.C; no longer IC2C.C
- net N$8: now also IC3D.C; no longer IC2D.C
Other:
- note added: "A"
- note added: "UniJoystiCle RETRO MOE"
- moved on the sheet: CN1, D1, IC2A, IC2B, IC2P, IC3A, IC3B, IC3P

Commit message: fix: board fixes
Parts:
- CN1: value 3.3V - 9V -> DC JACK; MF (none) -> SPC CONNECTORS; MPN (none) -> SPC21364; OC_NEWARK unknown -> 11M0559
- D1: value 1N4004 -> 1N4001; MF (none) -> NTE ELECTRONICS; MPN (none) -> 1N4001; OC_NEWARK unknown -> 10M8464
- IC1, IC2, IC3: MF (none) -> TEXAS INSTRUMENTS; MPN (none) -> SN74HC4066N; OC_NEWARK unknown -> 76C3574
- MOD1: value ESP12E_DEVKIT -> NodeMCU Amica v1.0
- X1: value Joy #1 -> DSUB 9; MF (none) -> FARNELL; MPN (none) -> 1-1634584-2; OC_NEWARK (none) -> 39K0552
- X2: value Joy #2 -> DSUB 9; MF (none) -> FARNELL; MPN (none) -> 1-1634584-2; OC_NEWARK (none) -> 39K0552
- renumbered ESP1 to MOD1
Changed lines of the file:
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@@
 </classes>
 <parts>
-<part name="ESP1" library="ESP12E_DEVKIT" deviceset="ESP12E_DEVKIT" device="">
+<part name="MOD1" library="ESP12E_DEVKIT" deviceset="ESP12E_DEVKIT" device="" value="NodeMCU Amica v1.0">
 <attribute name="MF" value=""/>
 <attribute name="MPN" value=""/>
 <attribute name="OC_NEWARK" value="unknown"/>
 </part>
-<part name="X1" library="con-subd" deviceset="F09" device="H" value="Joy #1"/>
-<part name="X2" library="con-subd" deviceset="F09" device="H" value="Joy #2"/>
+<part name="X1" library="con-subd" deviceset="F09" device="H" value="DSUB 9">
+<attribute name="MF" value="FARNELL"/>
+<attribute name="MPN" value="1-1634584-2"/>
+<attribute name="OC_NEWARK" value="39K0552"/>
+</part>
+<part name="X2" library="con-subd" deviceset="F09" device="H" value="DSUB 9">
+<attribute name="MF" value="FARNELL"/>
+<attribute name="MPN" value="1-1634584-2"/>
+<attribute name="OC_NEWARK" value="39K0552"/>
+</part>
 <part name="IC1" library="40xx" deviceset="4066" device="N">
-<attribute name="MF" value=""/>
-<attribute name="MPN" value=""/>
-<attribute name="OC_NEWARK" value="unknown"/>
+<attribute name="MF" value="TEXAS INSTRUMENTS"/>
+<attribute name="MPN" value="SN74HC4066N"/>
+<attribute name="OC_NEWARK" value="76C3574"/>
 </part>
 <part name="IC3" library="40xx" deviceset="4066" device="N">
-<attribute name="MF" value=""/>
-<attribute name="MPN" value=""/>
-<attribute name="OC_NEWARK" value="unknown"/>
+<attribute name="MF" value="TEXAS INSTRUMENTS"/>
+<attribute name="MPN" value="SN74HC4066N"/>
+<attribute name="OC_NEWARK" value="76C3574"/>
 </part>
 <part name="GND3" library="supply1" deviceset="GND" device=""/>
@@
 <part name="P+2" library="supply1" deviceset="VCC" device="" value="3.3v"/>
 <part name="IC2" library="40xx" deviceset="4066" device="N">
-<attribute name="MF" value=""/>
-<attribute name="MPN" value=""/>
-<attribute name="OC_NEWARK" value="unknown"/>
+<attribute name="MF" value="TEXAS INSTRUMENTS"/>
+<attribute name="MPN" value="SN74HC4066N"/>
+<attribute name="OC_NEWARK" value="76C3574"/>
 </part>
 <part name="FRAME1" library="frames" deviceset="LETTER_P" device="" value="Frame"/>
-<part name="CN1" library="adafruit" deviceset="DCBARREL" device="PTH" value="3.3V - 9V">
-<attribute name="MF" value=""/>
-<attribute name="MPN" value=""/>
-<attribute name="OC_NEWARK" value="unknown"/>
-</part>
-<part name="D1" library="diode" deviceset="1N4004" device="">
-<attribute name="MF" value=""/>
-<attribute name="MPN" value=""/>
-<attribute name="OC_NEWARK" value="unknown"/>
+<part name="CN1" library="adafruit" deviceset="DCBARREL" device="PTH" value="DC JACK">
+<attribute name="MF" value="SPC CONNECTORS"/>
+<attribute name="MPN" value="SPC21364"/>
+<attribute name="OC_NEWARK" value="11M0559"/>
+</part>
+<part name="D1" library="diode" deviceset="1N4004" device="" value="1N4001">
+<attribute name="MF" value="NTE ELECTRONICS"/>
+<attribute name="MPN" value="1N4001"/>
+<attribute name="OC_NEWARK" value="10M8464"/>
 </part>
 <part name="SUPPLY1" library="SparkFun-Aesthetics" deviceset="5V" device=""/>
@@
 </plain>
 <instances>
-<instance part="ESP1" gate="G$1" x="116.84" y="25.4" rot="R90">
+<instance part="MOD1" gate="G$1" x="116.84" y="25.4" rot="R90">
 <attribute name="OC_NEWARK" x="116.84" y="25.4" size="1.778" layer="96" display="off"/>
 <attribute name="MF" x="116.84" y="25.4" size="1.778" layer="96" display="off"/>
@@
 <net name="N$1" class="0">
 <segment>
-<pinref part="ESP1" gate="G$1" pin="D0"/>
+<pinref part="MOD1" gate="G$1" pin="D0"/>
 <wire x1="99.06" y1="43.18" x2="99.06" y2="48.26" width="0.1524" layer="91"/>
 <wire x1="99.06" y1="48.26" x2="22.86" y2="48.26" width="0.1524" layer="91"/>
@@
 <net name="N$2" class="0">
 <segment>
-<pinref part="ESP1" gate="G$1" pin="D1"/>
+<pinref part="MOD1" gate="G$1" pin="D1"/>
 <wire x1="101.6" y1="43.18" x2="101.6" y2="50.8" width="0.1524" layer="91"/>
 <wire x1="101.6" y1="50.8" x2="25.4" y2="50.8" width="0.1524" layer="91"/>
@@
 <net name="N$3" class="0">
 <segment>
-<pinref part="ESP1" gate="G$1" pin="D2"/>
+<pinref part="MOD1" gate="G$1" pin="D2"/>
 <wire x1="104.14" y1="43.18" x2="104.14" y2="53.34" width="0.1524" layer="91"/>
 <wire x1="104.14" y1="53.34" x2="27.94" y2="53.34" width="0.1524" layer="91"/>
@@
 <net name="N$4" class="0">
 <segment>
-<pinref part="ESP1" gate="G$1" pin="D3"/>
+<pinref part="MOD1" gate="G$1" pin="D3"/>
 <wire x1="106.68" y1="43.18" x2="106.68" y2="55.88" width="0.1524" layer="91"/>
 <wire x1="106.68" y1="55.88" x2="30.48" y2="55.88" width="0.1524" layer="91"/>
@@
 <net name="N$5" class="0">
 <segment>
-<pinref part="ESP1" gate="G$1" pin="D5"/>
+<pinref part="MOD1" gate="G$1" pin="D5"/>
 <wire x1="116.84" y1="43.18" x2="116.84" y2="137.16" width="0.1524" layer="91"/>
 <pinref part="IC3" gate="A" pin="C"/>
@@
 <net name="N$6" class="0">
 <segment>
-<pinref part="ESP1" gate="G$1" pin="D6"/>
+<pinref part="MOD1" gate="G$1" pin="D6"/>
 <wire x1="119.38" y1="43.18" x2="119.38" y2="119.38" width="0.1524" layer="91"/>
 <pinref part="IC3" gate="B" pin="C"/>
@@
 <net name="N$7" class="0">
 <segment>
-<pinref part="ESP1" gate="G$1" pin="D7"/>
+<pinref part="MOD1" gate="G$1" pin="D7"/>
 <wire x1="121.92" y1="43.18" x2="121.92" y2="101.6" width="0.1524" layer="91"/>
 <pinref part="IC3" gate="C" pin="C"/>
@@
 <net name="N$8" class="0">
 <segment>
-<pinref part="ESP1" gate="G$1" pin="D8"/>
+<pinref part="MOD1" gate="G$1" pin="D8"/>
 <wire x1="124.46" y1="43.18" x2="124.46" y2="83.82" width="0.1524" layer="91"/>
 <pinref part="IC3" gate="D" pin="C"/>
@@
 </segment>
 <segment>
-<pinref part="ESP1" gate="G$1" pin="GND@3"/>
+<pinref part="MOD1" gate="G$1" pin="GND@3"/>
 <wire x1="132.08" y1="43.18" x2="132.08" y2="55.88" width="0.1524" layer="91"/>
 <wire x1="132.08" y1="55.88" x2="137.16" y2="55.88" width="0.1524" layer="91"/>
@@
 </segment>
 <segment>
-<pinref part="ESP1" gate="G$1" pin="3V3@2"/>
+<pinref part="MOD1" gate="G$1" pin="3V3@2"/>
 <pinref part="P+1" gate="VCC" pin="VCC"/>
 <wire x1="134.62" y1="43.18" x2="144.78" y2="43.18" width="0.1524" layer="91"/>
@@
 <net name="N$19" class="0">
 <segment>
-<pinref part="ESP1" gate="G$1" pin="D4"/>
+<pinref part="MOD1" gate="G$1" pin="D4"/>
 <wire x1="109.22" y1="43.18" x2="109.22" y2="58.42" width="0.1524" layer="91"/>
 <wire x1="109.22" y1="58.42" x2="50.8" y2="58.42" width="0.1524" layer="91"/>
@@
 <net name="N$20" class="0">
 <segment>
-<pinref part="ESP1" gate="G$1" pin="RX"/>
+<pinref part="MOD1" gate="G$1" pin="RX"/>
 <wire x1="127" y1="43.18" x2="127" y2="66.04" width="0.1524" layer="91"/>
 <pinref part="IC2" gate="B" pin="C"/>
@@
 <segment>
 <pinref part="SUPPLY2" gate="G$1" pin="5V"/>
-<pinref part="ESP1" gate="G$1" pin="VIN"/>
+<pinref part="MOD1" gate="G$1" pin="VIN"/>
 <wire x1="139.7" y1="7.62" x2="134.62" y2="7.62" width="0.1524" layer="91"/>
 </segment>
@@
 </segment>
 <segment>
-<pinref part="ESP1" gate="G$1" pin="GND@1"/>
+<pinref part="MOD1" gate="G$1" pin="GND@1"/>
 <pinref part="GND2" gate="G$1" pin="3.3V"/>
 <wire x1="132.08" y1="0" x2="132.08" y2="7.62" width="0.1524" layer="91"/>
@@
 </sheet>
 </sheets>
+<errors>
+</errors>
 </schematic>
 </drawing>

Commit message: fix: new design
Parts:
- removed X1, X2: DSUB 9, con-subd:F09H
- added J1, J2: DB9, SparkFun-Connectors:DB9FEMALE
Connections:
- net N$10: now also J1.2; no longer X1.2
- net N$11: now also J1.3; no longer X1.3
- net N$12: now also J1.4; no longer X1.4
- net N$13: now also J2.1; no longer X2.1
- net N$14: now also J2.2; no longer X2.2
- net N$15: now also J2.3; no longer X2.3
- net N$16: now also J2.4; no longer X2.4
- net N$17: now also J1.8; no longer X1.8
- net N$18: now also J2.8; no longer X2.8
- net N$21: now also J1.6; no longer X1.6
- net N$22: now also J2.6; no longer X2.6
- net N$9: now also J1.1; no longer X1.1
Changed lines of the file:
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@@
 <attribute name="OC_NEWARK" value="unknown"/>
-</part>
-<part name="X1" library="con-subd" deviceset="F09" device="H" value="DSUB 9">
-<attribute name="MF" value="FARNELL"/>
-<attribute name="MPN" value="1-1634584-2"/>
-<attribute name="OC_NEWARK" value="39K0552"/>
-</part>
-<part name="X2" library="con-subd" deviceset="F09" device="H" value="DSUB 9">
-<attribute name="MF" value="FARNELL"/>
-<attribute name="MPN" value="1-1634584-2"/>
-<attribute name="OC_NEWARK" value="39K0552"/>
 </part>
 <part name="IC1" library="40xx" deviceset="4066" device="N">
@@
 <part name="GND1" library="SparkFun-Aesthetics" deviceset="GND2" device=""/>
 <part name="GND2" library="SparkFun-Aesthetics" deviceset="GND2" device=""/>
+<part name="J1" library="SparkFun-Connectors" deviceset="DB9" device="FEMALE" value="DB9">
+<attribute name="MF" value=""/>
+<attribute name="MPN" value="618009231121"/>
+<attribute name="OC_NEWARK" value="16T0655"/>
+</part>
+<part name="J2" library="SparkFun-Connectors" deviceset="DB9" device="FEMALE" value="DB9">
+<attribute name="MF" value=""/>
+<attribute name="MPN" value="618009231121"/>
+<attribute name="OC_NEWARK" value="16T0655"/>
+</part>
 </parts>
 <sheets>
@@
 <attribute name="MPN" x="116.84" y="25.4" size="1.778" layer="96" display="off"/>
 </instance>
-<instance part="X1" gate="G$1" x="68.58" y="172.72"/>
-<instance part="X2" gate="G$1" x="154.94" y="170.18"/>
 <instance part="IC1" gate="A" x="68.58" y="139.7">
 <attribute name="OC_NEWARK" x="68.58" y="139.7" size="1.778" layer="96" display="off"/>
@@
 <instance part="GND1" gate="G$1" x="66.04" y="15.24"/>
 <instance part="GND2" gate="G$1" x="132.08" y="-2.54"/>
+<instance part="J1" gate="G$1" x="68.58" y="172.72">
+<attribute name="OC_NEWARK" x="68.58" y="172.72" size="1.778" layer="96" display="off"/>
+<attribute name="MF" x="68.58" y="172.72" size="1.778" layer="96" display="off"/>
+<attribute name="MPN" x="68.58" y="172.72" size="1.778" layer="96" display="off"/>
+</instance>
+<instance part="J2" gate="G$1" x="154.94" y="170.18">
+<attribute name="OC_NEWARK" x="154.94" y="170.18" size="1.778" layer="96" display="off"/>
+<attribute name="MF" x="154.94" y="170.18" size="1.778" layer="96" display="off"/>
+<attribute name="MPN" x="154.94" y="170.18" size="1.778" layer="96" display="off"/>
+</instance>
 </instances>
 <busses>
@@
 <net name="N$9" class="0">
 <segment>
-<pinref part="X1" gate="G$1" pin="1"/>
 <wire x1="60.96" y1="177.8" x2="53.34" y2="177.8" width="0.1524" layer="91"/>
 <wire x1="53.34" y1="177.8" x2="53.34" y2="142.24" width="0.1524" layer="91"/>
 <pinref part="IC1" gate="A" pin="A"/>
 <wire x1="53.34" y1="142.24" x2="55.88" y2="142.24" width="0.1524" layer="91"/>
+<pinref part="J1" gate="G$1" pin="1"/>
 </segment>
 </net>
 <net name="N$10" class="0">
 <segment>
-<pinref part="X1" gate="G$1" pin="2"/>
 <wire x1="60.96" y1="175.26" x2="50.8" y2="175.26" width="0.1524" layer="91"/>
 <wire x1="50.8" y1="175.26" x2="50.8" y2="124.46" width="0.1524" layer="91"/>
 <pinref part="IC1" gate="B" pin="A"/>
 <wire x1="50.8" y1="124.46" x2="55.88" y2="124.46" width="0.1524" layer="91"/>
+<pinref part="J1" gate="G$1" pin="2"/>
 </segment>
 </net>
 <net name="N$11" class="0">
 <segment>
-<pinref part="X1" gate="G$1" pin="3"/>
 <wire x1="60.96" y1="172.72" x2="48.26" y2="172.72" width="0.1524" layer="91"/>
 <wire x1="48.26" y1="172.72" x2="48.26" y2="106.68" width="0.1524" layer="91"/>
 <pinref part="IC1" gate="C" pin="A"/>
 <wire x1="48.26" y1="106.68" x2="55.88" y2="106.68" width="0.1524" layer="91"/>
+<pinref part="J1" gate="G$1" pin="3"/>
 </segment>
 </net>
 <net name="N$12" class="0">
 <segment>
-<pinref part="X1" gate="G$1" pin="4"/>
 <wire x1="60.96" y1="170.18" x2="45.72" y2="170.18" width="0.1524" layer="91"/>
 <wire x1="45.72" y1="170.18" x2="45.72" y2="88.9" width="0.1524" layer="91"/>
 <pinref part="IC1" gate="D" pin="A"/>
 <wire x1="45.72" y1="88.9" x2="55.88" y2="88.9" width="0.1524" layer="91"/>
+<pinref part="J1" gate="G$1" pin="4"/>
 </segment>
 </net>
 <net name="N$13" class="0">
 <segment>
-<pinref part="X2" gate="G$1" pin="1"/>
 <wire x1="147.32" y1="175.26" x2="139.7" y2="175.26" width="0.1524" layer="91"/>
 <wire x1="139.7" y1="175.26" x2="139.7" y2="142.24" width="0.1524" layer="91"/>
 <pinref part="IC3" gate="A" pin="A"/>
 <wire x1="139.7" y1="142.24" x2="142.24" y2="142.24" width="0.1524" layer="91"/>
+<pinref part="J2" gate="G$1" pin="1"/>
 </segment>
 </net>
 <net name="N$14" class="0">
 <segment>
-<pinref part="X2" gate="G$1" pin="2"/>
 <wire x1="147.32" y1="172.72" x2="137.16" y2="172.72" width="0.1524" layer="91"/>
 <wire x1="137.16" y1="172.72" x2="137.16" y2="124.46" width="0.1524" layer="91"/>
 <pinref part="IC3" gate="B" pin="A"/>
 <wire x1="137.16" y1="124.46" x2="142.24" y2="124.46" width="0.1524" layer="91"/>
+<pinref part="J2" gate="G$1" pin="2"/>
 </segment>
 </net>
 <net name="N$15" class="0">
 <segment>
-<pinref part="X2" gate="G$1" pin="3"/>
 <wire x1="147.32" y1="170.18" x2="134.62" y2="170.18" width="0.1524" layer="91"/>
 <wire x1="134.62" y1="170.18" x2="134.62" y2="106.68" width="0.1524" layer="91"/>
 <pinref part="IC3" gate="C" pin="A"/>
 <wire x1="134.62" y1="106.68" x2="142.24" y2="106.68" width="0.1524" layer="91"/>
+<pinref part="J2" gate="G$1" pin="3"/>
 </segment>
 </net>
 <net name="N$16" class="0">
 <segment>
-<pinref part="X2" gate="G$1" pin="4"/>
 <wire x1="147.32" y1="167.64" x2="132.08" y2="167.64" width="0.1524" layer="91"/>
 <wire x1="132.08" y1="167.64" x2="132.08" y2="88.9" width="0.1524" layer="91"/>
 <pinref part="IC3" gate="D" pin="A"/>
 <wire x1="132.08" y1="88.9" x2="142.24" y2="88.9" width="0.1524" layer="91"/>
+<pinref part="J2" gate="G$1" pin="4"/>
 </segment>
 </net>
 <net name="N$17" class="0">
 <segment>
-<pinref part="X1" gate="G$1" pin="8"/>
 <wire x1="76.2" y1="170.18" x2="83.82" y2="170.18" width="0.1524" layer="91"/>
 <wire x1="83.82" y1="170.18" x2="83.82" y2="142.24" width="0.1524" layer="91"/>
@@
 <pinref part="IC2" gate="A" pin="B"/>
 <wire x1="83.82" y1="71.12" x2="81.28" y2="71.12" width="0.1524" layer="91"/>
+<pinref part="J1" gate="G$1" pin="8"/>
 </segment>
 </net>
 <net name="N$18" class="0">
 <segment>
-<pinref part="X2" gate="G$1" pin="8"/>
 <wire x1="162.56" y1="167.64" x2="170.18" y2="167.64" width="0.1524" layer="91"/>
 <wire x1="170.18" y1="167.64" x2="170.18" y2="142.24" width="0.1524" layer="91"/>
@@
 <pinref part="IC2" gate="B" pin="B"/>
 <wire x1="170.18" y1="71.12" x2="167.64" y2="71.12" width="0.1524" layer="91"/>
+<pinref part="J2" gate="G$1" pin="8"/>
 </segment>
 </net>
@@
 <net name="N$21" class="0">
 <segment>
-<pinref part="X1" gate="G$1" pin="6"/>
 <wire x1="76.2" y1="175.26" x2="76.2" y2="185.42" width="0.1524" layer="91"/>
 <wire x1="76.2" y1="185.42" x2="38.1" y2="185.42" width="0.1524" layer="91"/>
@@
 <pinref part="IC2" gate="A" pin="A"/>
 <wire x1="38.1" y1="71.12" x2="55.88" y2="71.12" width="0.1524" layer="91"/>
+<pinref part="J1" gate="G$1" pin="6"/>
 </segment>
 </net>
@@
 <wire x1="129.54" y1="182.88" x2="165.1" y2="182.88" width="0.1524" layer="91"/>
 <wire x1="165.1" y1="182.88" x2="165.1" y2="172.72" width="0.1524" layer="91"/>
-<pinref part="X2" gate="G$1" pin="6"/>
 <wire x1="165.1" y1="172.72" x2="162.56" y2="172.72" width="0.1524" layer="91"/>
-</segment>
-</net>
+<pinref part="J2" gate="G$1" pin="6"/>
+</segment>
+</net>
